Commit message: Makes a 3 Joint robot

File: body.urdf (robot description, URDF)
Before this commit: robot robot, 7 links, 6 joints
Links:
- removed link 0
- removed link 1
- removed link 2
- removed link 3
- removed link 4
- removed link 5
- removed link 6
- added link BackLeg, mass 1; collision box size=1 1 1; visual box size=1 1 1
- added link FrontLeg, mass 1; collision box size=1 1 1; visual box size=1 1 1
- added link Torso, mass 1; collision box size=1 1 1; visual box size=1 1 1
Joints:
- removed joint 0_1
- removed joint 1_2
- removed joint 2_3
- removed joint 3_4
- removed joint 4_5
- removed joint 5_6
- added joint BackLeg_Torso: type revolute, parent BackLeg, child Torso, origin xyz=1.0 0 1.0 rpy=0 0 0, axis 0 1 0, limit lower=-3.14159 upper=3.14159 effort=0.0 velocity=0.0
- added joint Torso_FrontLeg: type revolute, parent Torso, child FrontLeg, origin xyz=1 0 0 rpy=0 0 0, axis 0 1 0, limit lower=-3.14159 upper=3.14159 effort=0.0 velocity=0.0
